File: sharkpad rev2.kicad_pcb (KiCad board)
At the start: 2 copper layers, 80.2 x 78 mm, 55 parts, among them J1 USB C, SW1 Z, SW2 TAC1, SW3 X, SW4 TAC2, SW5 C, SW6 TAC3, SW7 EC11E15244G1, U1 RP2040, U2 XC6206, U3 SRV05-4, U4 W25Q128JVS, Y1 12MHz

Commit message: remove leds from bom, move jumper to side of board
Parts:
- moved JP1 18.3 mm to (147.9, 115.3)
Routing:
- net /~{BOOTSEL}: track 2.28 -> 20.3 mm, vias 0 -> 2
- net GND: track 57.9 -> 56.1 mm, vias 34 -> 33
- net /COL1: track 67.1 -> 67.9 mm
Changed lines of the file:
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@@
     (property "Sheetfile" "sharkpad rev2.kicad_sch")
     (property "Sheetname" "")
-    (attr smd)
+    (property "exclude_from_bom" "")
+    (attr smd exclude_from_pos_files exclude_from_bom)
     (fp_text reference "LED2" (at 3.8 0) (layer "B.SilkS") hide
       (effects (font (size 1 1) (thickness 0.15)) (justify left mirror))
@@
     (property "Sheetfile" "sharkpad rev2.kicad_sch")
     (property "Sheetname" "")
-    (attr smd)
+    (property "exclude_from_bom" "")
+    (attr smd exclude_from_pos_files exclude_from_bom)
     (fp_text reference "LED3" (at 3.8 0) (layer "B.SilkS") hide
       (effects (font (size 1 1) (thickness 0.15)) (justify left mirror))
@@
     (property "Sheetfile" "sharkpad rev2.kicad_sch")
     (property "Sheetname" "")
-    (attr smd)
+    (property "exclude_from_bom" "")
+    (attr smd exclude_from_pos_files exclude_from_bom)
     (fp_text reference "LED1" (at 3.8 0) (layer "B.SilkS") hide
       (effects (font (size 1 1) (thickness 0.15)) (justify left mirror))
@@
     (descr "LED SMD 0603 (1608 Metric), square (rectangular) end terminal, IPC_7351 nominal, (Body size source: http://www.tortai-tech.com/upload/download/2011102023233369053.pdf), generated with kicad-footprint-generator")
     (tags "LED")
+    (property "LCSC" "C72043")
     (property "Sheetfile" "sharkpad rev2.kicad_sch")
     (property "Sheetname" "")
@@
   )
   (footprint "Jumper:SolderJumper-2_P1.3mm_Open_Pad1.0x1.5mm" (layer "B.Cu")
-    (at 129.6 115.3 -90)
+    (at 147.9 115.3 -90)
     (descr "SMD Solder Jumper, 1x1.5mm Pads, 0.3mm gap, open")
     (tags "solder jumper open")
@@
     (property "exclude_from_bom" "")
     (attr exclude_from_pos_files exclude_from_bom)
-    (fp_text reference "JP1" (at 0 1.8 -270) (layer "B.SilkS") hide
-      (effects (font (size 1 1) (thickness 0.15)) (justify mirror))
-    )
-    (fp_text value "BOOTSEL" (at 0 -1.9 -270) (layer "B.Fab")
+    (fp_text reference "JP1" (at 0 1.8 90) (layer "B.SilkS") hide
+      (effects (font (size 1 1) (thickness 0.15)) (justify mirror))
+    )
+    (fp_text value "BOOTSEL" (at 0 -1.9 90) (layer "B.Fab")
       (effects (font (size 1 1) (thickness 0.15)) (justify mirror))
     )
@@
   (via (at 109.7 114.6) (size 1) (drill 0.6) (layers "F.Cu" "B.Cu") (net 1))
   (via (at 110.9 65.5) (size 1) (drill 0.6) (layers "F.Cu" "B.Cu") (net 1))
-  (via (at 129.6 112.8) (size 1) (drill 0.6) (layers "F.Cu" "B.Cu") (net 1))
   (via (at 90.1 92.5) (size 1) (drill 0.6) (layers "F.Cu" "B.Cu") (net 1))
   (via (at 89.4 71.4) (size 1) (drill 0.6) (layers "F.Cu" "B.Cu") (net 1))
@@
   (segment (start 122.5375 70.1625) (end 122.6 70.1) (width 0.5) (layer "B.Cu") (net 1))
   (segment (start 109.445 112.02) (end 109.445 111.145) (width 0.5) (layer "B.Cu") (net 1))
-  (segment (start 129.6 114.65) (end 129.6 112.8) (width 0.5) (layer "B.Cu") (net 1))
   (segment (start 128.43 92.53) (end 128.4 92.5) (width 0.5) (layer "B.Cu") (net 1))
   (segment (start 117.35 64.0505) (end 117.4995 64.2) (width 0.5) (layer "B.Cu") (net 1))
@@
   (via (at 133.7 119.7) (size 0.8) (drill 0.4) (layers "F.Cu" "B.Cu") (net 10))
   (via (at 124.9 102.5) (size 0.8) (drill 0.4) (layers "F.Cu" "B.Cu") (net 10))
+  (segment (start 131.7 102.4) (end 136.3625 102.4) (width 0.25) (layer "B.Cu") (net 10))
+  (segment (start 139.7625 102.6) (end 137.9625 100.8) (width 0.25) (layer "B.Cu") (net 10))
   (segment (start 142.5 102.9) (end 142.2 102.6) (width 0.25) (layer "B.Cu") (net 10))
-  (segment (start 131.7 102.4) (end 136.3625 102.4) (width 0.25) (layer "B.Cu") (net 10))
   (segment (start 137.9625 100.8) (end 136.3625 102.4) (width 0.25) (layer "B.Cu") (net 10))
+  (segment (start 135.4 118) (end 135.4 113.2) (width 0.25) (layer "B.Cu") (net 10))
   (segment (start 118.2 120.4) (end 118.5 120.7) (width 0.2) (layer "B.Cu") (net 10))
   (segment (start 118.9 100.8) (end 120.6 102.5) (width 0.25) (layer "B.Cu") (net 10))
-  (segment (start 142.2 102.6) (end 139.7625 102.6) (width 0.25) (layer "B.Cu") (net 10))
+  (segment (start 133.7 119.7) (end 135.4 118) (width 0.25) (layer "B.Cu") (net 10))
   (segment (start 130.1 100.8) (end 128.425 100.8) (width 0.25) (layer "B.Cu") (net 10))
-  (segment (start 133.7 119.7) (end 133.7 114.9) (width 0.25) (layer "B.Cu") (net 10))
   (segment (start 131.7 102.4) (end 130.1 100.8) (width 0.25) (layer "B.Cu") (net 10))
   (segment (start 120.6 102.5) (end 124.9 102.5) (width 0.25) (layer "B.Cu") (net 10))
+  (segment (start 117.5375 120.4) (end 118.2 120.4) (width 0.2) (layer "B.Cu") (net 10))
+  (segment (start 142.2 102.6) (end 139.7625 102.6) (width 0.25) (layer "B.Cu") (net 10))
+  (segment (start 118.5 120.7) (end 129.1 120.7) (width 0.2) (layer "B.Cu") (net 10))
   (segment (start 142.5 106.1) (end 142.5 102.9) (width 0.25) (layer "B.Cu") (net 10))
-  (segment (start 117.5375 120.4) (end 118.2 120.4) (width 0.2) (layer "B.Cu") (net 10))
-  (segment (start 118.5 120.7) (end 129.1 120.7) (width 0.2) (layer "B.Cu") (net 10))
-  (segment (start 139.7625 102.6) (end 137.9625 100.8) (width 0.25) (layer "B.Cu") (net 10))
-  (segment (start 133.7 114.9) (end 142.5 106.1) (width 0.25) (layer "B.Cu") (net 10))
+  (segment (start 135.4 113.2) (end 142.5 106.1) (width 0.25) (layer "B.Cu") (net 10))
   (segment (start 119.35 82.28) (end 119.35 79.2) (width 0.25) (layer "B.Cu") (net 11))
   (segment (start 125.075 104.7) (end 131.575 104.7) (width 0.25) (layer "F.Cu") (net 12))
@@
   (segment (start 109.78 61.73) (end 109.78 57.55) (width 0.25) (layer "B.Cu") (net 22))
   (segment (start 109.78 57.55) (end 118.42 57.55) (width 0.25) (layer "B.Cu") (net 22))
-  (segment (start 128.31 117.7) (end 129.355 116.655) (width 0.5) (layer "B.Cu") (net 23))
-  (segment (start 129.6 116.41) (end 129.6 115.95) (width 0.5) (layer "B.Cu") (net 23))
-  (segment (start 129.355 116.655) (end 129.6 116.41) (width 0.5) (layer "B.Cu") (net 23))
+  (segment (start 139.075 117.675) (end 139.1 117.7) (width 0.25) (layer "F.Cu") (net 23))
+  (segment (start 130 117.7) (end 130.025 117.675) (width 0.25) (layer "F.Cu") (net 23))
+  (segment (start 130.025 117.675) (end 139.075 117.675) (width 0.25) (layer "F.Cu") (net 23))
+  (via (at 139.1 117.7) (size 0.8) (drill 0.4) (layers "F.Cu" "B.Cu") (net 23))
+  (via (at 130 117.7) (size 0.8) (drill 0.4) (layers "F.Cu" "B.Cu") (net 23))
+  (segment (start 139.1 117.7) (end 146.15 117.7) (width 0.25) (layer "B.Cu") (net 23))
+  (segment (start 128.31 117.7) (end 130 117.7) (width 0.25) (layer "B.Cu") (net 23))
+  (segment (start 146.15 117.7) (end 147.9 115.95) (width 0.25) (layer "B.Cu") (net 23))
   (segment (start 112.3 121.6375) (end 112.3 122.169975) (width 0.2) (layer "B.Cu") (net 24))
   (segment (start 111.669975 122.8) (end 110.19 122.8) (width 0.2) (layer "B.Cu") (net 24))
@@
   (segment (start 87.7 101.6) (end 104.1 118) (width 0.2) (layer "B.Cu") (net 28))
   (segment (start 104.1 118) (end 110.6625 118) (width 0.2) (layer "B.Cu") (net 28))
-  (segment (start 130.5 119.6) (end 129.1 119.6) (width 0.25) (layer "F.Cu") (net 29))
   (segment (start 110.29 95.19) (end 110.29 85.66) (width 0.25) (layer "F.Cu") (net 29))
+  (segment (start 131.9 119.6) (end 129.1 119.6) (width 0.25) (layer "F.Cu") (net 29))
   (segment (start 131.575 100.2) (end 133.1 101.725) (width 0.25) (layer "F.Cu") (net 29))
   (segment (start 122.475 97.6) (end 112.7 97.6) (width 0.25) (layer "F.Cu") (net 29))
   (segment (start 125.075 100.2) (end 122.475 97.6) (width 0.25) (layer "F.Cu") (net 29))
+  (segment (start 133.1 118.4) (end 131.9 119.6) (width 0.25) (layer "F.Cu") (net 29))
   (segment (start 112.7 97.6) (end 110.29 95.19) (width 0.25) (layer "F.Cu") (net 29))
-  (segment (start 133.1 114.3) (end 133.1 117) (width 0.25) (layer "F.Cu") (net 29))
-  (segment (start 133.1 117) (end 130.5 119.6) (width 0.25) (layer "F.Cu") (net 29))
   (segment (start 125.075 100.2) (end 131.575 100.2) (width 0.25) (layer "F.Cu") (net 29))
   (segment (start 133.1 101.725) (end 133.1 103.3) (width 0.25) (layer "F.Cu") (net 29))
   (via (at 129.1 119.6) (size 0.8) (drill 0.4) (layers "F.Cu" "B.Cu") (net 29))
   (via (at 133.1 103.3) (size 0.8) (drill 0.4) (layers "F.Cu" "B.Cu") (net 29))
-  (via (at 133.1 114.3) (size 0.8) (drill 0.4) (layers "F.Cu" "B.Cu") (net 29))
-  (segment (start 133.1 103.3) (end 133.1 114.3) (width 0.25) (layer "B.Cu") (net 29))
+  (via (at 133.1 118.4) (size 0.8) (drill 0.4) (layers "F.Cu" "B.Cu") (net 29))
   (segment (start 117.5375 120) (end 121.2 120) (width 0.2) (layer "B.Cu") (net 29))
+  (segment (start 133.1 103.3) (end 133.1 118.4) (width 0.25) (layer "B.Cu") (net 29))
   (segment (start 121.6 119.6) (end 129.1 119.6) (width 0.2) (layer "B.Cu") (net 29))
   (segment (start 121.2 120) (end 121.6 119.6) (width 0.2) (layer "B.Cu") (net 29))

Commit message: nothing changes
Parts:
- added kibuzzard-638A2C0C: G***, kibuzzard-638A2C0C, B.Cu at (117.5, 71.2)
- added kibuzzard-638A2C3F: G***, kibuzzard-638A2C3F, B.Cu at (117.1, 77.2)
- added kibuzzard-638A2CDC: G***, kibuzzard-638A2CDC, B.Cu at (147.9, 117.9)
- added kibuzzard-638A2DF9: G***, kibuzzard-638A2DF9, B.Cu at (114.0, 73.5)
- turned REF** to 90 degrees
Routing:
- net /RGB_UNDERGLOW: track 33.7 -> 34.3 mm
Other:
- board text added: "JLCJLCJLCJLC"

Commit message: rev2 first draft
Parts:
- added kibuzzard-5: G***, kibuzzard-638B4E2B, B.Cu at (92.6, 102.7)
- added kibuzzard-6: G***, kibuzzard-638B4E4E, B.Cu at (92.6, 109.0)
- SW2: renamed from SW6; footprint Button_Switch_THT:SW_PUSH_6mm_H8mm -> Button_Switch_THT:SW_PUSH_6mm_H13mm
- SW3: renamed from SW4; footprint Button_Switch_THT:SW_PUSH_6mm_H8mm -> Button_Switch_THT:SW_PUSH_6mm_H13mm
- SW4: renamed from SW2; footprint Button_Switch_THT:SW_PUSH_6mm_H8mm -> Button_Switch_THT:SW_PUSH_6mm_H13mm
- renumbered C14 to C1, C7 to C10, C3 to C11, C6 to C12, C10 to C13, C5 to C14, C12 to C15, C15 to C16, C13 to C17, C11 to C2, C16 to C3, C9 to C4, C17 to C5, C4 to C6, C1 to C7, C2 to C8, C8 to C9, D9 to D1, D6 to D2, D1 to D3, D7 to D4, D3 to D5, D10 to D6, D2 to D7, D11 to D8, LED3 to LED1, LED1 to LED3, R7 to R1, R5 to R2, R6 to R3, R3 to R5, R2 to R6, R8 to R7, R1 to R8, SW7 to SW1, SW3 to SW6, SW1 to SW7, U2 to U1, U4 to U2, U1 to U4, kibuzzard-638A2CDC to kibuzzard-1, kibuzzard-638A2C3F to kibuzzard-2, kibuzzard-638A2C0C to kibuzzard-3, kibuzzard-638A2DF9 to kibuzzard-4
Routing:
- net GND: track 56.1 -> 80.5 mm, vias 33 -> 40
- net /COL0: track 85.5 -> 93.0 mm
- net /ROW0: track 105.6 -> 111.4 mm
- net /COL3: track 76.4 -> 79.7 mm
- net /ROTB: track 66.3 -> 67.8 mm
- net /ROW1: track 67.0 -> 67.6 mm
- net +5V: track 89.0 -> 89.6 mm
- net /QSPI_CS: track 16.5 -> 16.0 mm

Commit message: rev2 draft 2
Parts:
- removed D3: LED_Small, LED_SMD:LED_0603_1608Metric
- removed R1: 1k, Resistor_SMD:R_0402_1005Metric
- removed kibuzzard-4: G***, kibuzzard-638A2DF9
- JP1: footprint Jumper:SolderJumper-2_P1.3mm_Open_Pad1.0x1.5mm -> Connector_PinHeader_2.54mm:PinHeader_1x02_P2.54mm_Vertical
- moved kibuzzard-2 3.40 mm to (116.2, 73.9)
- moved JP1 0.78 mm to (148.7, 115.3), turned to 90 degrees
- moved kibuzzard-1 0.50 mm to (147.4, 117.9)
Routing:
- net /PWR_LED_A: track 1.71 -> 0.00 mm
- net GND: track 80.5 -> 79.0 mm, vias 40 -> 39
- net /~{BOOTSEL}: track 20.3 -> 18.8 mm
- net +3V3: track 175.1 -> 173.6 mm

Commit message: finish
Parts:
- JP1: footprint Connector_PinHeader_2.54mm:PinHeader_1x02_P2.54mm_Vertical -> marbastlib-various:SW_SPST_SKQG_WithStem
- moved JP1 3.30 mm to (148.5, 112.0)
- moved kibuzzard-1 1.13 mm to (148.5, 117.6)
Routing:
- net /~{BOOTSEL}: track 18.8 -> 25.6 mm
