File: sharkpad rev2.kicad_sch (KiCad schematic)
At the start: 51 parts, among them J1 USB C, SW1 Z, SW2 TAC1, SW3 X, SW4 TAC2, SW5 C, SW6 TAC3, SW7 EC11E15244G1, U1 RP2040, U2 XC6206, U3 SRV05-4, U4 W25Q128JVS, Y1 12MHz

Commit message: remove leds from bom, move jumper to side of board
Parts:
- LED1, LED2, LED3: now left out of the parts list
Changed lines of the file:
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@@
   )
   (symbol (lib_id "marbastlib-mx:MX_SK6812MINI-E") (at 262.89 31.75 0) (unit 1)
-    (in_bom yes) (on_board yes) (fields_autoplaced)
+    (in_bom no) (on_board yes) (fields_autoplaced)
     (property "Reference" "LED1" (id 0) (at 265.43 25.4 0))
     (property "Value" "SK6812MINI-E" (id 1) (at 276.86 29.9593 0)
@@
   )
   (symbol (lib_id "marbastlib-mx:MX_SK6812MINI-E") (at 262.89 64.77 0) (unit 1)
-    (in_bom yes) (on_board yes)
+    (in_bom no) (on_board yes)
     (property "Reference" "LED2" (id 0) (at 265.43 58.42 0))
     (property "Value" "SK6812MINI-E" (id 1) (at 276.86 62.9793 0)
@@
   )
   (symbol (lib_id "marbastlib-mx:MX_SK6812MINI-E") (at 262.89 97.79 0) (unit 1)
-    (in_bom yes) (on_board yes)
+    (in_bom no) (on_board yes) (fields_autoplaced)
     (property "Reference" "LED3" (id 0) (at 265.43 91.44 0))
     (property "Value" "SK6812MINI-E" (id 1) (at 276.86 95.9993 0)

Commit message: rev2 first draft
Parts:
- SW2: renamed from SW6; footprint Button_Switch_THT:SW_PUSH_6mm_H8mm -> Button_Switch_THT:SW_PUSH_6mm_H13mm
- SW3: renamed from SW4; footprint Button_Switch_THT:SW_PUSH_6mm_H8mm -> Button_Switch_THT:SW_PUSH_6mm_H13mm
- SW4: renamed from SW2; footprint Button_Switch_THT:SW_PUSH_6mm_H8mm -> Button_Switch_THT:SW_PUSH_6mm_H13mm
- renumbered C14 to C1, C7 to C10, C3 to C11, C6 to C12, C10 to C13, C5 to C14, C12 to C15, C15 to C16, C13 to C17, C11 to C2, C16 to C3, C9 to C4, C17 to C5, C4 to C6, C1 to C7, C2 to C8, C8 to C9, D9 to D1, D6 to D2, D1 to D3, D7 to D4, D3 to D5, D10 to D6, D2 to D7, D11 to D8, LED3 to LED1, LED1 to LED3, R7 to R1, R5 to R2, R6 to R3, R3 to R5, R2 to R6, R8 to R7, R1 to R8, SW7 to SW1, SW3 to SW6, SW1 to SW7, U2 to U1, U4 to U2, U1 to U4
Other:
- note added: "In-key RGB LEDs"
- note added: "Key Matrix"
- note added: "QSPI Flash"
- note added: "RP2040 and Crystal"
- note added: "USB-C Port, ESD, and 3.3v LDO"
- moved on the sheet: C3, D1, D2, D4, D5, D6, D7, D8, JP1, R3, SW1, SW2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

Commit message: rev2 draft 2
Parts:
- removed D3: LED_Small, LED_SMD:LED_0603_1608Metric, symbol Device:LED_Small
- removed R1: 1k, Resistor_SMD:R_0402_1005Metric, symbol Device:R_Small
- JP1: footprint Jumper:SolderJumper-2_P1.3mm_Open_Pad1.0x1.5mm -> Connector_PinHeader_2.54mm:PinHeader_1x02_P2.54mm_Vertical
Changed lines of the file:
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@@
   (junction (at 251.46 154.94) (diameter 0) (color 0 0 0 0)
   )
-  (junction (at 165.1 33.02) (diameter 0) (color 0 0 0 0)
-  )
   (junction (at 71.12 153.67) (diameter 0) (color 0 0 0 0)
   )
@@
   )
   (junction (at 160.02 33.02) (diameter 0) (color 0 0 0 0)
-  )
-  (junction (at 160.02 40.64) (diameter 0) (color 0 0 0 0)
   )
   (junction (at 53.34 153.67) (diameter 0) (color 0 0 0 0)
@@
     (stroke (width 0) (type default) (color 0 0 0 0))
   )
-  (wire (pts (xy 175.26 33.02) (xy 175.26 40.64))
-    (stroke (width 0) (type default) (color 0 0 0 0))
-  )
   (wire (pts (xy 101.6 210.82) (xy 109.22 210.82))
     (stroke (width 0) (type default) (color 0 0 0 0))
@@
     (stroke (width 0) (type default) (color 0 0 0 0))
   )
-  (wire (pts (xy 173.99 33.02) (xy 175.26 33.02))
-    (stroke (width 0) (type default) (color 0 0 0 0))
-  )
   (wire (pts (xy 78.74 153.67) (xy 78.74 154.94))
     (stroke (width 0) (type default) (color 0 0 0 0))
@@
     (stroke (width 0) (type default) (color 0 0 0 0))
   )
-  (wire (pts (xy 160.02 40.64) (xy 168.91 40.64))
-    (stroke (width 0) (type default) (color 0 0 0 0))
-  )
   (polyline (pts (xy 195.58 218.44) (xy 266.7 218.44))
     (stroke (width 0) (type default) (color 0 0 0 0))
@@
     (stroke (width 0) (type default) (color 0 0 0 0))
   )
-  (wire (pts (xy 175.26 40.64) (xy 173.99 40.64))
-    (stroke (width 0) (type default) (color 0 0 0 0))
-  )
   (wire (pts (xy 77.47 39.37) (xy 77.47 41.91))
     (stroke (width 0) (type default) (color 0 0 0 0))
@@
   )
   (wire (pts (xy 273.05 165.1) (xy 289.56 165.1))
-    (stroke (width 0) (type default) (color 0 0 0 0))
-  )
-  (wire (pts (xy 165.1 33.02) (xy 168.91 33.02))
     (stroke (width 0) (type default) (color 0 0 0 0))
   )
@@
   (label "QSPI_SD2" (at 38.1 190.5 0)
     (effects (font (size 1.27 1.27)) (justify left bottom))
-  )
-  (label "PWR_LED_A" (at 175.26 40.64 90)
-    (effects (font (size 0.5 0.5)) (justify left bottom))
   )
   (label "D_+" (at 46.99 170.18 0)
@@
     )
     (property "LCSC" "C52923" (id 4) (at 137.16 35.5662 0)
-      (effects (font (size 1.27 1.27)) hide)
-    )
-    (pin "1")
-    (pin "2")
-  )
-  (symbol (lib_id "Device:LED_Small") (at 171.45 40.64 0) (unit 1)
-    (in_bom yes) (on_board yes) (fields_autoplaced)
-    (property "Reference" "D3" (id 0) (at 171.5135 36.83 0))
-    (property "Value" "LED_Small" (id 1) (at 171.5135 36.83 0)
-      (effects (font (size 1.27 1.27)) hide)
-    )
-    (property "Footprint" "LED_SMD:LED_0603_1608Metric" (id 2) (at 171.45 40.64 90)
-      (effects (font (size 1.27 1.27)) hide)
-    )
-    (property "Datasheet" "~" (id 3) (at 171.45 40.64 90)
-      (effects (font (size 1.27 1.27)) hide)
-    )
-    (property "LCSC" "C72043" (id 4) (at 171.5135 36.83 0)
       (effects (font (size 1.27 1.27)) hide)
     )
@@
       (effects (font (size 1.27 1.27)) hide)
     )
-    (property "Footprint" "Jumper:SolderJumper-2_P1.3mm_Open_Pad1.0x1.5mm" (id 2) (at 167.64 259.08 0)
+    (property "Footprint" "Connector_PinHeader_2.54mm:PinHeader_1x02_P2.54mm_Vertical" (id 2) (at 167.64 259.08 0)
       (effects (font (size 1.27 1.27)) hide)
     )
@@
     (pin "2")
   )
-  (symbol (lib_id "Device:R_Small") (at 171.45 33.02 90) (unit 1)
-    (in_bom yes) (on_board yes)
-    (property "Reference" "R1" (id 0) (at 171.45 30.48 90))
-    (property "Value" "1k" (id 1) (at 175.26 31.75 90))
-    (property "Footprint" "Resistor_SMD:R_0402_1005Metric" (id 2) (at 171.45 33.02 0)
-      (effects (font (size 1.27 1.27)) hide)
-    )
-    (property "Datasheet" "~" (id 3) (at 171.45 33.02 0)
-      (effects (font (size 1.27 1.27)) hide)
-    )
-    (property "LCSC" "C11702" (id 4) (at 171.45 30.48 0)
-      (effects (font (size 1.27 1.27)) hide)
-    )
-    (pin "1")
-    (pin "2")
-  )
   (symbol (lib_id "Device:C_Small") (at 24.13 218.44 90) (unit 1)
     (in_bom yes) (on_board yes)
@@
       (reference "D2") (unit 1) (value "D_Small") (footprint "Diode_SMD:D_SOD-123")
     )
-    (path "/2e03a152-ec32-4f76-9550-903f5e61f1ee"
-      (reference "D3") (unit 1) (value "LED_Small") (footprint "LED_SMD:LED_0603_1608Metric")
-    )
     (path "/9bc9f9b7-d4fe-49c1-857f-4e08e226a2fc"
       (reference "D4") (unit 1) (value "D_Small") (footprint "Diode_SMD:D_SOD-123")
@@
     )
     (path "/d0573173-b83b-4023-89e7-ab4ec45892d3"
-      (reference "JP1") (unit 1) (value "BOOTSEL") (footprint "Jumper:SolderJumper-2_P1.3mm_Open_Pad1.0x1.5mm")
+      (reference "JP1") (unit 1) (value "BOOTSEL") (footprint "Connector_PinHeader_2.54mm:PinHeader_1x02_P2.54mm_Vertical")
     )
     (path "/4bdb33ac-1e13-4242-90da-b2029f01a98b"
@@
       (reference "LED3") (unit 1) (value "SK6812MINI-E") (footprint "marbastlib-mx:LED_MX_6028R-FLIPPED")
     )
-    (path "/d1d82d21-d316-411f-9436-75f9bad9e137"
-      (reference "R1") (unit 1) (value "1k") (footprint "Resistor_SMD:R_0402_1005Metric")
-    )
     (path "/ba40aee3-9605-4b69-ad21-5d85be0a110c"

Commit message: finish
Parts:
- JP1: footprint Connector_PinHeader_2.54mm:PinHeader_1x02_P2.54mm_Vertical -> marbastlib-various:SW_SPST_SKQG_WithStem; now in the parts list
